File: hardware/PicoROM-32/PicoROM.kicad_pcb (KiCad board)
At the start: 6 copper layers, 42.2 x 17.8 mm, 56 parts, among them J1 USB_C_Receptacle_USB2.0, J2 External Reset, J3 Conn_01x16, J4 Conn_01x16, J5 Conn_01x05_Pin, U1 AP2112K-3.3, U10 74LVCH8T245, U2 W25Q16JVUXIQ, U3 RP2040, U4 74LVCH245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

Commit message: Hardware reorg
Parts:
- U10: footprint RP2040_minimal:DHVQFN24_L5.5-W3.5-P0.50-BL-EP -> PicoROM:DHVQFN24_L5.5-W3.5-P0.50-BL-EP
- U3: footprint RP2040_minimal:RP2040-QFN-56 -> PicoROM:RP2040-QFN-56
- U4, U5, U9: footprint RP2040_minimal:V-QFN4525-20_L4.5-W2.5-P0.50-BL -> PicoROM:V-QFN4525-20_L4.5-W2.5-P0.50-BL
- U7: footprint RP2040_minimal:X2QFN-8_L1.5-W1.5-P0.50-BL -> PicoROM:X2QFN-8_L1.5-W1.5-P0.50-BL
Changed lines of the file:
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@@
 		)
 	)
-	(footprint "RP2040_minimal:RP2040-QFN-56"
+	(footprint "PicoROM:RP2040-QFN-56"
 		(layer "F.Cu")
 		(at 95.693122 63.319035 -135)
@@
 			)
 		)
-		(property "Footprint" "RP2040_minimal:RP2040-QFN-56"
+		(property "Footprint" "PicoROM:RP2040-QFN-56"
 			(at 0 0 -135)
 			(unlocked yes)
@@
 			)
 		)
-		(model "3dshapes/USON-8_L2-W3-H0.6X0.5P.wrl"
+		(model "../3dshapes/USON-8_L2-W3-H0.6X0.5P.wrl"
 			(offset
 				(xyz 0 0 0)
@@
 			)
 		)
-		(model "3dshapes/USB-C-SMD_GT-USB-7051A.wrl"
+		(model "../3dshapes/USB-C-SMD_GT-USB-7051A.wrl"
 			(offset
 				(xyz 0 0 6.3)
@@
 		)
 	)
-	(footprint "RP2040_minimal:DHVQFN24_L5.5-W3.5-P0.50-BL-EP"
+	(footprint "PicoROM:DHVQFN24_L5.5-W3.5-P0.50-BL-EP"
 		(layer "F.Cu")
 		(at 87.295 67.9 -90)
@@
 			)
 		)
-		(property "Footprint" "RP2040_minimal:DHVQFN24_L5.5-W3.5-P0.50-BL-EP"
+		(property "Footprint" "PicoROM:DHVQFN24_L5.5-W3.5-P0.50-BL-EP"
 			(at 0 0 90)
 			(layer "F.Fab")
@@
 			(layers "F.Cu" "F.Paste" "F.Mask")
 		)
-		(model "3dshapes/DHVQFN24_L5.5-W3.5-H0.9-P0.50-BL-EP.wrl"
+		(model "../3dshapes/DHVQFN24_L5.5-W3.5-H0.9-P0.50-BL-EP.wrl"
 			(offset
 				(xyz 0 -0 -0)
@@
 		)
 	)
-	(footprint "RP2040_minimal:X2QFN-8_L1.5-W1.5-P0.50-BL"
+	(footprint "PicoROM:X2QFN-8_L1.5-W1.5-P0.50-BL"
 		(layer "F.Cu")
 		(at 105.06 59.8 180)
@@
 			)
 		)
-		(property "Footprint" "RP2040_minimal:X2QFN-8_L1.5-W1.5-P0.50-BL"
+		(property "Footprint" "PicoROM:X2QFN-8_L1.5-W1.5-P0.50-BL"
 			(at 0 0 360)
 			(layer "F.Fab")
@@
 			(pintype "unspecified+no_connect")
 		)
-		(model "3dshapes/X2QFN-8_L1.5-W1.5-P0.50-BL.wrl"
+		(model "../3dshapes/X2QFN-8_L1.5-W1.5-P0.50-BL.wrl"
 			(offset
 				(xyz 0.01 0.02 -0)
@@
 		)
 	)
-	(footprint "RP2040_minimal:V-QFN4525-20_L4.5-W2.5-P0.50-BL"
+	(footprint "PicoROM:V-QFN4525-20_L4.5-W2.5-P0.50-BL"
 		(layer "B.Cu")
 		(at 105.345 60.8375 180)
@@
 			)
 		)
-		(property "Footprint" "RP2040_minimal:V-QFN4525-20_L4.5-W2.5-P0.50-BL"
+		(property "Footprint" "PicoROM:V-QFN4525-20_L4.5-W2.5-P0.50-BL"
 			(at 0 0 0)
 			(layer "B.Fab")
@@
 			(layers "B.Cu" "B.Paste" "B.Mask")
 		)
-		(model "3dshapes/V-QFN4525-20_L4.5-W2.5-P0.50-BL.wrl"
+		(model "../3dshapes/V-QFN4525-20_L4.5-W2.5-P0.50-BL.wrl"
 			(offset
 				(xyz 0 -0 -0)
@@
 		)
 	)
-	(footprint "RP2040_minimal:V-QFN4525-20_L4.5-W2.5-P0.50-BL"
+	(footprint "PicoROM:V-QFN4525-20_L4.5-W2.5-P0.50-BL"
 		(layer "B.Cu")
 		(at 110.245 64.5 90)
@@
 			)
 		)
-		(property "Footprint" "RP2040_minimal:V-QFN4525-20_L4.5-W2.5-P0.50-BL"
+		(property "Footprint" "PicoROM:V-QFN4525-20_L4.5-W2.5-P0.50-BL"
 			(at 0 0 90)
 			(layer "B.Fab")
@@
 			(layers "B.Cu" "B.Paste" "B.Mask")
 		)
-		(model "3dshapes/V-QFN4525-20_L4.5-W2.5-P0.50-BL.wrl"
+		(model "../3dshapes/V-QFN4525-20_L4.5-W2.5-P0.50-BL.wrl"
 			(offset
 				(xyz 0 -0 -0)
@@
 		)
 	)
-	(footprint "RP2040_minimal:V-QFN4525-20_L4.5-W2.5-P0.50-BL"
+	(footprint "PicoROM:V-QFN4525-20_L4.5-W2.5-P0.50-BL"
 		(layer "B.Cu")
 		(at 105.47 68.4)
@@
 			)
 		)
-		(property "Footprint" "RP2040_minimal:V-QFN4525-20_L4.5-W2.5-P0.50-BL"
+		(property "Footprint" "PicoROM:V-QFN4525-20_L4.5-W2.5-P0.50-BL"
 			(at 0 0 360)
 			(layer "B.Fab")
@@
 			(layers "B.Cu" "B.Paste" "B.Mask")
 		)
-		(model "3dshapes/V-QFN4525-20_L4.5-W2.5-P0.50-BL.wrl"
+		(model "../3dshapes/V-QFN4525-20_L4.5-W2.5-P0.50-BL.wrl"
 			(offset
 				(xyz 0 -0 -0)
