File: hardware/PicoROM-32/PicoROM.kicad_sch (KiCad schematic)
At the start: 56 parts, among them J1 USB_C_Receptacle_USB2.0, J2 External Reset, J3 Conn_01x16, J4 Conn_01x16, J5 Conn_01x05_Pin, U1 AP2112K-3.3, U10 74LVCH8T245, U2 W25Q16JVUXIQ, U3 RP2040, U4 74LVCH245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

Commit message: Hardware reorg
Parts:
- U10: footprint RP2040_minimal:DHVQFN24_L5.5-W3.5-P0.50-BL-EP -> PicoROM:DHVQFN24_L5.5-W3.5-P0.50-BL-EP
- U3: footprint RP2040_minimal:RP2040-QFN-56 -> PicoROM:RP2040-QFN-56
- U4, U5, U9: footprint RP2040_minimal:V-QFN4525-20_L4.5-W2.5-P0.50-BL -> PicoROM:V-QFN4525-20_L4.5-W2.5-P0.50-BL
- U7: footprint RP2040_minimal:X2QFN-8_L1.5-W1.5-P0.50-BL -> PicoROM:X2QFN-8_L1.5-W1.5-P0.50-BL
Changed lines of the file:
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@@
 			)
 		)
-		(property "Footprint" "RP2040_minimal:RP2040-QFN-56"
+		(property "Footprint" "PicoROM:RP2040-QFN-56"
 			(at 179.07 144.78 0)
 			(effects
@@
 			)
 		)
-		(property "Footprint" "RP2040_minimal:X2QFN-8_L1.5-W1.5-P0.50-BL"
+		(property "Footprint" "PicoROM:X2QFN-8_L1.5-W1.5-P0.50-BL"
 			(at 328.93 133.35 0)
 			(effects
@@
 			)
 		)
-		(property "Footprint" "RP2040_minimal:V-QFN4525-20_L4.5-W2.5-P0.50-BL"
+		(property "Footprint" "PicoROM:V-QFN4525-20_L4.5-W2.5-P0.50-BL"
 			(at 69.85 238.76 0)
 			(effects
@@
 			)
 		)
-		(property "Footprint" "RP2040_minimal:V-QFN4525-20_L4.5-W2.5-P0.50-BL"
+		(property "Footprint" "PicoROM:V-QFN4525-20_L4.5-W2.5-P0.50-BL"
 			(at 110.49 238.76 0)
 			(effects
@@
 			)
 		)
-		(property "Footprint" "RP2040_minimal:DHVQFN24_L5.5-W3.5-P0.50-BL-EP"
+		(property "Footprint" "PicoROM:DHVQFN24_L5.5-W3.5-P0.50-BL-EP"
 			(at 269.24 255.27 0)
 			(effects
@@
 			)
 		)
-		(property "Footprint" "RP2040_minimal:V-QFN4525-20_L4.5-W2.5-P0.50-BL"
+		(property "Footprint" "PicoROM:V-QFN4525-20_L4.5-W2.5-P0.50-BL"
 			(at 154.94 238.76 0)
 			(effects
