File: hardware/PicoROM/PicoROM.kicad_sch (KiCad schematic)
At the start: 61 parts, among them J1 USB_C_Receptacle_USB2.0, J2 External Reset, J3 Conn_01x16, J4 Conn_01x16, J5 Conn_01x05_Pin, U1 NCP114AMX330TCG, U10 74LVC8245, U2 W25Q16JVUXIQ, U3 RP2040, U4 74LVC245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

Commit message: Created new 32-pin version from 28-pin version
Parts:
- removed C26, C27: 1u, Capacitor_SMD:C_0402_1005Metric, symbol Device:C
- removed R14, R29: 1k, Resistor_SMD:R_0201_0603Metric, symbol Device:R
- removed U1, U8: NCP114AMX330TCG, Package_DFN_QFN:OnSemi_XDFN4-1EP_1.0x1.0mm_EP0.52x0.52mm, symbol Regulator_Linear:NCP115AMX250TCG
- removed U6: 74LVC2G125, Package_SO:VSSOP-8_2.3x2mm_P0.5mm, symbol 74xGxx:74LVC2G125
- removed U7: 74LVC1G32, PicoROM:USON-6_L1.5-W1.0-P0.50-BL, symbol 74xGxx:74LVC1G32
- added U1: AP2112K-3.3, Package_TO_SOT_SMD:SOT-23-5, symbol Regulator_Linear:AP2112K-3.3
- added U7: TCA5405RUGR, PicoROM:X2QFN-8_L1.5-W1.5-P0.50-BL, symbol TCA5404:TCA5405RUGR
- added U8: 74AHCT1G126, Package_TO_SOT_SMD:SOT-23-5, symbol 74xGxx:74AHCT1G126
- C1, C4: footprint Capacitor_SMD:C_0402_1005Metric -> Capacitor_SMD:C_0805_2012Metric; MPN C52923 -> C28323
- D1: footprint LED_SMD:LED_0402_1005Metric -> LED_SMD:LED_0603_1608Metric; MPN C434450 -> C510027
- D2: footprint LED_SMD:LED_0402_1005Metric -> LED_SMD:LED_0603_1608Metric; MPN C71911 -> C2922668
- D3: footprint LED_SMD:LED_0402_1005Metric -> LED_SMD:LED_0603_1608Metric; MPN C434450 -> C2925173
- J2: footprint Connector_PinHeader_2.54mm:PinHeader_1x02_P2.54mm_Vertical -> Connector_PinHeader_2.54mm:PinHeader_1x01_P2.54mm_Vertical; symbol Connector:Conn_01x02_Pin -> Connector:Conn_01x01_Pin
- J3, J4: now left out of the parts list
- J5: footprint Connector_PinHeader_1.27mm:PinHeader_1x05_P1.27mm_Vertical -> Connector_PinHeader_1.00mm:PinHeader_1x05_P1.00mm_Vertical
- R11: value 1k -> 100k; MPN C270335 -> C270364
- U10: value 74LVC8245 -> 74LVCH8T245; MPN C548858 -> C458263
- U4, U5, U9: value 74LVC245 -> 74LVCH245; MPN C2676234 -> C548916
Connections:
- net +3V3_SYS is gone; now on net +3V3: C19.1, C20.1, C21.1, C23.1, C24.1, R11.2, U10.23 (VCCB), U10.24 (VCCB), U4.20 (VCC), U5.20 (VCC), U9.20 (VCC)
- net ~{EXT_RESET_EN} is gone; now on net D6: U3.40 (GPIO28_ADC2)
- net +3V3: now also U1.5 (VOUT), U7.1 (VCC)
- net +5V: now also C18.1, C22.1, C25.1, U10.1 (VCCA), U1.1 (VIN), U1.3 (EN), U8.5 (VCC)
- net D0: now also U3.34 (GPIO22); no longer U3.29 (GPIO18)
- net D1: now also U3.35 (GPIO23); no longer U3.30 (GPIO19)
- net D2: now also U3.36 (GPIO24); no longer U3.31 (GPIO20)
- net D3: now also U3.37 (GPIO25); no longer U3.32 (GPIO21)
- net D4: now also U3.38 (GPIO26_ADC0); no longer U3.34 (GPIO22)
- net D5: now also U3.39 (GPIO27_ADC1); no longer U3.35 (GPIO23)
- net D6: no longer U3.36 (GPIO24)
- net D7: now also U3.41 (GPIO29_ADC3); no longer U3.37 (GPIO25)
- net GND: now also U10.22 (~{OE}), U1.2 (GND), U7.3 (GND), U8.3 (GND); no longer U10.2 (DIR), U4.14 (B4), U4.15 (B3), U4.16 (B2), U5.15 (B3), U5.16 (B2), U5.18 (B0)
- net INFO_LED1: now also U7.6 (Q2); no longer U3.41 (GPIO29_ADC3)
- net ~{BUF_OE}: now also U10.2 (DIR), U3.30 (GPIO19); no longer U10.22 (~{OE}), U3.39 (GPIO27_ADC1)
- net ~{OE}: now also U3.31 (GPIO20), U5.4 (A2); no longer U3.38 (GPIO26_ADC0)
- net ~{PIN_CE}: now also R11.1, U5.18 (B0)
- net ~{PIN_OE}: now also U5.16 (B2)
- net INFO_LED2: now reaches R2.2
- net INFO_LED2: now also U7.7 (Q3)
- net at R8.2: now also U8.4
- net at D3.2 (A): now also R2.1; no longer R11.1
- net ~{CE}: now reaches U5.2 (A0)
- net ~{CE}: now also U3.32 (GPIO21)
- removed net +5V_SYS: C18.1, C22.1, C25.1, D5.2 (A), J4.1 (Pin_1), U10.1 (VCCA)
- net EXT_RESET_HIGH renamed EXT_RESET
- net EXT_RESET: now also R8.1; no longer R2.1
- removed net EXT_RESET_LOW: J2.2 (Pin_2), R8.1
- new net EXT_RESET_EN: U7.4 (Q0), U8.1
- new net EXT_RESET_VALUE: U7.5 (Q1), U8.2
- new net IO_EXPAND: U3.29 (GPIO18), U7.2 (DIN)
- new net PIN_5V: D5.2 (A), J4.1 (Pin_1)
- no-connect marks 11 -> 14
Other:
- note added: "IOs"
- note removed: "Input Buffers"
- note removed: "Output Buffer"
- title: PicoROM-32 - ROM Emulator -> PicoROM - ROM Emulator
- moved on the sheet: C1, C18, C19, C2, C20, C22, C23, C24, C25, C3, C4, C5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
